Commit message: add world frame

File: 3Dperception_ws/src/robot_description/urdf/robot.urdf.xacro (robot description, xacro)
@@ -3,5 +3,13 @@
   <xacro:include filename="$(find robot_description)/urdf/common_properties.xacro"/>
   <xacro:include filename="$(find robot_description)/urdf/robot.gazebo.xacro"/>
+  <!--Links-->
+  <link name="world"/>
   <link name="base_footprint"/>
+  <!-- Joints -->
+  <joint name="world_joint" type="fixed">
+    <origin xyz="0 0 0" rpy="0 0 0" />
+    <child link="base_footprint" />
+    <parent link="world"/>
+  </joint>
   <joint name="base_joint" type="fixed">
     <parent link="base_footprint"/>
