Commit message: update robot

File: 3Dperception_ws/src/robot/urdf/robot.gazebo.xacro (robot description, xacro)
@@ -1,4 +1,4 @@
 <?xml version="1.0"?>
-<robot name="robot_sim" xmlns:xacro="http://ros.org/wiki/xacro">
+<robot name="turtlebot3_waffle_pi_sim" xmlns:xacro="http://ros.org/wiki/xacro">
   <xacro:arg name="laser_visual"  default="false"/>
   <xacro:arg name="camera_visual" default="false"/>
@@ -53,5 +53,5 @@
   </gazebo>
   <gazebo>
-    <plugin name="robot_controller" filename="libgazebo_ros_diff_drive.so">
+    <plugin name="turtlebot3_waffle_pi_controller" filename="libgazebo_ros_diff_drive.so">
       <commandTopic>cmd_vel</commandTopic>
       <odometryTopic>odom</odometryTopic>

File: 3Dperception_ws/src/robot/urdf/robot.urdf.xacro (robot description, xacro)
@@ -1,15 +1,15 @@
 <?xml version="1.0" ?>
 <robot name="robot" xmlns:xacro="http://ros.org/wiki/xacro">
-  <xacro:include filename="$(find robot_description)/urdf/common_properties.xacro"/>
-  <xacro:include filename="$(find robot_description)/urdf/robot.gazebo.xacro"/>
+  <xacro:include filename="$(find robot)/urdf/common_properties.xacro"/>
+  <xacro:include filename="$(find robot)/urdf/robot.gazebo.xacro"/>
   <!--Links-->
-  <link name="world"/>
+  <!-- <link name="world"/> -->
   <link name="base_footprint"/>
   <!-- Joints -->
-  <joint name="world_joint" type="fixed">
+  <!-- <joint name="world_joint" type="fixed">
     <origin xyz="0 0 0" rpy="0 0 0" />
     <child link="base_footprint" />
     <parent link="world"/>
-  </joint>
+  </joint> -->
   <joint name="base_joint" type="fixed">
     <parent link="base_footprint"/>
@@ -21,5 +21,5 @@
       <origin xyz="-0.064 0 0.0" rpy="0 0 0"/>
       <geometry>
-        <mesh filename="package://robot_description/meshes/bases/waffle_pi_base.stl" scale="0.001 0.001 0.001"/>
+        <mesh filename="package://robot/meshes/bases/waffle_pi_base.stl" scale="0.001 0.001 0.001"/>
       </geometry>
       <material name="light_black"/>
@@ -49,5 +49,5 @@
       <origin xyz="0 0 0" rpy="1.57 0 0"/>
       <geometry>
-        <mesh filename="package://robot_description/meshes/wheels/left_tire.stl" scale="0.001 0.001 0.001"/>
+        <mesh filename="package://robot/meshes/wheels/left_tire.stl" scale="0.001 0.001 0.001"/>
       </geometry>
       <material name="dark"/>
@@ -77,5 +77,5 @@
       <origin xyz="0 0 0" rpy="1.57 0 0"/>
       <geometry>
-        <mesh filename="package://robot_description/meshes/wheels/right_tire.stl" scale="0.001 0.001 0.001"/>
+        <mesh filename="package://robot/meshes/wheels/right_tire.stl" scale="0.001 0.001 0.001"/>
       </geometry>
       <material name="dark"/>
@@ -135,5 +135,5 @@
     </inertial>
   </link>
-  <joint name="imu_joint" type="fixed">
+  <!-- <joint name="imu_joint" type="fixed">
     <parent link="base_link"/>
     <child link="imu_link"/>
@@ -150,5 +150,5 @@
       <origin xyz="0 0 0.0" rpy="0 0 0"/>
       <geometry>
-        <mesh filename="package://robot_description/meshes/sensors/lds.stl" scale="0.001 0.001 0.001"/>
+        <mesh filename="package://robot/meshes/sensors/lds.stl" scale="0.001 0.001 0.001"/>
       </geometry>
       <material name="dark"/>
@@ -167,5 +167,5 @@
                izz="0.001" />
     </inertial>
-  </link>
+  </link> -->
   <joint name="camera_joint" type="fixed">
     <origin xyz="0.073 -0.011 0.084" rpy="0 0 0"/>
