Commit message: add camera shaft mount and camera to robot model

File: 3Dperception_ws/src/robot/urdf/robot.urdf.xacro (robot description, xacro)
@@ -3,4 +3,5 @@
   <xacro:include filename="$(find robot)/urdf/common_properties.xacro"/>
   <xacro:include filename="$(find robot)/urdf/robot.gazebo.xacro"/>
+  <xacro:include filename="$(find realsense2_camera)/urdf/_d435.urdf.xacro"/>
   <!--Links-->
   <!-- <link name="world"/> -->
@@ -168,28 +169,34 @@
     </inertial>
   </link> -->
-  <joint name="camera_joint" type="fixed">
-    <origin xyz="0.073 -0.011 0.084" rpy="0 0 0"/>
-    <parent link="base_link"/>
-    <child link="camera_link"/>
-  </joint>
-  <link name="camera_link">
-    <collision>
-      <origin xyz="0.005 0.011 0.013" rpy="0 0 0"/>
-      <geometry>
-        <box size="0.015 0.030 0.027"/>
-      </geometry>
-    </collision>
-  </link>
-  <joint name="camera_rgb_joint" type="fixed">
-    <origin xyz="0.003 0.011 0.009" rpy="0 0 0"/>
-    <parent link="camera_link"/>
-    <child link="camera_rgb_frame"/>
-  </joint>
-  <link name="camera_rgb_frame"/>
-  <joint name="camera_rgb_optical_joint" type="fixed">
-    <origin xyz="0 0 0" rpy="-1.57 0 -1.57"/>
-    <parent link="camera_rgb_frame"/>
-    <child link="camera_rgb_optical_frame"/>
-  </joint>
-  <link name="camera_rgb_optical_frame"/>
+  <joint name="base_to_camera_shaft_joint" type="fixed">
+    <origin xyz="0.0 0.0 0.092" rpy="0 0 0"/>
+    <parent link="base_link"/>
+    <child link="camera_shaft_link"/>
+  </joint>
+  <link name="camera_shaft_link">
+    <visual>
+      <origin xyz="0 0 0.092" rpy="0 0 0" />
+      <geometry>
+        <box size="0.02 0.02 0.2"/>
+      </geometry>
+      <material name="white"/>
+    </visual>
+  </link>
+  <joint name="camera_shaft_to_camera_joint" type="fixed">
+    <origin xyz="0.02 0.0 0.17" rpy="0 0.4 0"/>
+    <parent link="camera_shaft_link"/>
+    <child link="camera_mount_link"/>
+  </joint>
+  <link name="camera_mount_link">
+    <visual>
+      <origin xyz="0.0 0.0 0.0" rpy="0 0 0"/>
+      <geometry>
+        <box size="0.02 0.02 0.02"/>
+      </geometry>
+      <material name="black"/>
+    </visual>
+  </link>
+  <sensor_d435 parent="camera_mount_link">
+    <origin xyz="0 0 0.01" rpy="0 0 0"/>
+  </sensor_d435>
 </robot>

Commit message: update urdf

File: 3Dperception_ws/src/robot/urdf/robot.urdf.xacro (robot description, xacro)
@@ -7,4 +7,5 @@
   <!-- <link name="world"/> -->
   <link name="base_footprint"/>
+  <link name="front_base_footprint"/>
   <!-- Joints -->
   <!-- <joint name="world_joint" type="fixed">
@@ -18,4 +19,9 @@
     <origin xyz="0 0 0.010" rpy="0 0 0"/>
   </joint>
+  <joint name="front_base_joint" type="fixed">
+    <parent link="base_footprint"/>
+    <child link="front_base_footprint" />
+    <origin xyz="-0.19 0 0" rpy="0 0 -3.147"/>
+  </joint>
   <link name="base_link">
     <visual>
@@ -170,13 +176,13 @@
   </link> -->
   <joint name="base_to_camera_shaft_joint" type="fixed">
-    <origin xyz="0.0 0.0 0.092" rpy="0 0 0"/>
-    <parent link="base_link"/>
+    <origin xyz="-0.115 0.0 0.126" rpy="0 0 0"/>
+    <parent link="front_base_footprint"/>
     <child link="camera_shaft_link"/>
   </joint>
   <link name="camera_shaft_link">
     <visual>
-      <origin xyz="0 0 0.092" rpy="0 0 0" />
-      <geometry>
-        <box size="0.02 0.02 0.2"/>
+      <origin xyz="0 0 0.126" rpy="0 0 0" />
+      <geometry>
+        <box size="0.02 0.02 0.30"/>
       </geometry>
       <material name="white"/>
@@ -184,5 +190,6 @@
   </link>
   <joint name="camera_shaft_to_camera_joint" type="fixed">
-    <origin xyz="0.02 0.0 0.17" rpy="0 0.4 0"/>
+    <origin xyz="0.02 0.0 0.24" rpy="0 0.35 0"/>
+    <!-- <origin xyz="0.02 0.0 0.42" rpy="0 0.6 0"/> -->
     <parent link="camera_shaft_link"/>
     <child link="camera_mount_link"/>

Commit message: update urdf according to new camera position

File: 3Dperception_ws/src/robot/urdf/robot.urdf.xacro (robot description, xacro)
@@ -190,5 +190,5 @@
   </link>
   <joint name="camera_shaft_to_camera_joint" type="fixed">
-    <origin xyz="0.02 0.0 0.24" rpy="0 0.35 0"/>
+    <origin xyz="0.02 0.0 0.27" rpy="0 0.315 0"/>
     <!-- <origin xyz="0.02 0.0 0.42" rpy="0 0.6 0"/> -->
     <parent link="camera_shaft_link"/>

Commit message: New hyper parameters and post processing criteria

File: 3Dperception_ws/src/robot/urdf/robot.urdf.xacro (robot description, xacro)
@@ -22,5 +22,5 @@
     <parent link="base_footprint"/>
     <child link="front_base_footprint" />
-    <origin xyz="-0.19 0 0" rpy="0 0 -3.147"/>
+    <origin xyz="0.064 0 0" rpy="0 0 0"/>
   </joint>
   <link name="base_link">
@@ -46,4 +46,14 @@
     </inertial>
   </link>
+  <joint name="tray_joint" type="fixed">
+    <origin xyz="0.4 0.0 0.0" rpy="0 0 0"/>
+    <parent link="front_base_footprint"/>
+    <child link="tray_front_link"/>
+  </joint>
+  <link name="tray_front_link">
+    <visual>
+      <origin xyz="0.4 0.0 0.0" rpy="0 0 0"/>
+    </visual>
+  </link>
   <joint name="wheel_left_joint" type="continuous">
     <parent link="base_link"/>
@@ -190,5 +200,5 @@
   </link>
   <joint name="camera_shaft_to_camera_joint" type="fixed">
-    <origin xyz="0.02 0.0 0.27" rpy="0 0.315 0"/>
+    <origin xyz="0.02 0.0 0.25" rpy="0 0.35 0"/>
     <!-- <origin xyz="0.02 0.0 0.42" rpy="0 0.6 0"/> -->
     <parent link="camera_shaft_link"/>
